File: H1DR51/Design/H1DR51.sch (EAGLE design)
At the start: 39 parts, among them J1 WURTH_74980111211WURTH_749801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, P1 HEXABIT_17.32_NO_P6_P7_P12, U1 STM32G0B1CEU6NUFQFPN48_STM32_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, U2 ENC28J60-I/SSSSOP28_MC_MCH, X1 XTALL_CSTCE8M00G52, X2 25.0 MHz

Commit message: -Correct some documentaion issues
Connections:
- net USART2_RX: now also P1.SD2; no longer P1.SD5
- net USART2_TX: now also P1.SU2; no longer P1.SU5
- net USART3_RX: now also P1.SD3; no longer P1.SD1
- net USART3_TX: now also P1.SU3; no longer P1.SU1
- net USART4_RX: now also P1.SD1; no longer P1.SD4
- net USART4_TX: now also P1.SU1; no longer P1.SU4
- net USART5_RX: now also P1.SD4; no longer P1.SD2
- net USART5_TX: now also P1.SU4; no longer P1.SU2
- net USART6_RX: now also P1.SD5; no longer P1.SD3
- net USART6_TX: now also P1.SU5; no longer P1.SU3
Other:
- note removed: "P1"
- note removed: "P2*"
- note removed: "P3"
- note removed: "P4"
- note removed: "P5"
Changed lines of the file:
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@@
 <?xml version="1.0" encoding="utf-8"?>
 <!DOCTYPE eagle SYSTEM "eagle.dtd">
-<eagle version="9.6.2">
+<eagle version="9.6.1">
 <drawing>
 <settings>
@@
 <text x="243.84" y="146.05" size="1.778" layer="95">BOOT</text>
 <text x="179.4328" y="4.9414" size="1.9304" layer="101" font="vector">Obada Albasha</text>
-<text x="53.34" y="151.765" size="1.27" layer="95">P2*</text>
-<text x="53.34" y="156.845" size="1.27" layer="95">P1</text>
-<text x="53.34" y="161.925" size="1.27" layer="95">P5</text>
-<text x="53.34" y="167.005" size="1.27" layer="95">P4</text>
-<text x="53.34" y="172.085" size="1.27" layer="95">P3</text>
-<text x="53.34" y="116.205" size="1.27" layer="95">P2*</text>
-<text x="53.34" y="121.285" size="1.27" layer="95">P1</text>
-<text x="53.34" y="126.365" size="1.27" layer="95">P5</text>
-<text x="53.34" y="131.445" size="1.27" layer="95">P4</text>
-<text x="53.34" y="136.525" size="1.27" layer="95">P3</text>
 </plain>
 <instances>
@@
 </segment>
 <segment>
-<pinref part="P1" gate="G$1" pin="SD2"/>
-<wire x1="67.945" y1="132.08" x2="81.915" y2="132.08" width="0.1524" layer="91"/>
-<label x="68.58" y="132.715" size="1.778" layer="95"/>
+<pinref part="P1" gate="G$1" pin="SD4"/>
+<wire x1="67.945" y1="121.92" x2="81.915" y2="121.92" width="0.1524" layer="91"/>
+<label x="68.58" y="122.555" size="1.778" layer="95"/>
 </segment>
 </net>
@@
 </segment>
 <segment>
-<pinref part="P1" gate="G$1" pin="SU2"/>
-<wire x1="67.945" y1="167.64" x2="81.915" y2="167.64" width="0.1524" layer="91"/>
-<label x="67.945" y="168.275" size="1.778" layer="95"/>
+<pinref part="P1" gate="G$1" pin="SU4"/>
+<wire x1="67.945" y1="157.48" x2="81.915" y2="157.48" width="0.1524" layer="91"/>
+<label x="67.945" y="158.115" size="1.778" layer="95"/>
 </segment>
 </net>
@@
 </segment>
 <segment>
-<pinref part="P1" gate="G$1" pin="SU4"/>
-<wire x1="67.945" y1="157.48" x2="81.915" y2="157.48" width="0.1524" layer="91"/>
-<label x="67.945" y="158.115" size="1.778" layer="95"/>
+<pinref part="P1" gate="G$1" pin="SU1"/>
+<wire x1="67.945" y1="172.72" x2="81.915" y2="172.72" width="0.1524" layer="91"/>
+<label x="67.945" y="173.355" size="1.778" layer="95"/>
 </segment>
 </net>
@@
 </segment>
 <segment>
-<pinref part="P1" gate="G$1" pin="SD4"/>
-<wire x1="67.945" y1="121.92" x2="81.915" y2="121.92" width="0.1524" layer="91"/>
-<label x="68.58" y="122.555" size="1.778" layer="95"/>
+<pinref part="P1" gate="G$1" pin="SD1"/>
+<wire x1="67.945" y1="137.16" x2="81.915" y2="137.16" width="0.1524" layer="91"/>
+<label x="68.58" y="137.795" size="1.778" layer="95"/>
 </segment>
 </net>
@@
 </segment>
 <segment>
-<pinref part="P1" gate="G$1" pin="SU5"/>
-<wire x1="67.945" y1="152.4" x2="81.915" y2="152.4" width="0.1524" layer="91"/>
-<label x="67.945" y="153.035" size="1.778" layer="95"/>
+<pinref part="P1" gate="G$1" pin="SU2"/>
+<wire x1="67.945" y1="167.64" x2="81.915" y2="167.64" width="0.1524" layer="91"/>
+<label x="67.945" y="168.275" size="1.778" layer="95"/>
 </segment>
 </net>
@@
 </segment>
 <segment>
-<pinref part="P1" gate="G$1" pin="SD5"/>
-<wire x1="67.945" y1="116.84" x2="81.915" y2="116.84" width="0.1524" layer="91"/>
-<label x="68.58" y="117.475" size="1.778" layer="95"/>
+<pinref part="P1" gate="G$1" pin="SD2"/>
+<wire x1="67.945" y1="132.08" x2="81.915" y2="132.08" width="0.1524" layer="91"/>
+<label x="68.58" y="132.715" size="1.778" layer="95"/>
 </segment>
 </net>
@@
 </segment>
 <segment>
-<pinref part="P1" gate="G$1" pin="SU1"/>
-<wire x1="67.945" y1="172.72" x2="81.915" y2="172.72" width="0.1524" layer="91"/>
-<label x="67.945" y="173.355" size="1.778" layer="95"/>
+<pinref part="P1" gate="G$1" pin="SU3"/>
+<wire x1="67.945" y1="162.56" x2="81.915" y2="162.56" width="0.1524" layer="91"/>
+<label x="67.945" y="163.195" size="1.778" layer="95"/>
 </segment>
 </net>
@@
 </segment>
 <segment>
-<pinref part="P1" gate="G$1" pin="SD1"/>
-<wire x1="67.945" y1="137.16" x2="81.915" y2="137.16" width="0.1524" layer="91"/>
-<label x="68.58" y="137.795" size="1.778" layer="95"/>
+<pinref part="P1" gate="G$1" pin="SD3"/>
+<wire x1="67.945" y1="127" x2="81.915" y2="127" width="0.1524" layer="91"/>
+<label x="68.58" y="127.635" size="1.778" layer="95"/>
 </segment>
 </net>
@@
 </segment>
 <segment>
-<pinref part="P1" gate="G$1" pin="SD3"/>
-<wire x1="67.945" y1="127" x2="81.915" y2="127" width="0.1524" layer="91"/>
-<label x="68.58" y="127.635" size="1.778" layer="95"/>
+<pinref part="P1" gate="G$1" pin="SD5"/>
+<wire x1="67.945" y1="116.84" x2="81.915" y2="116.84" width="0.1524" layer="91"/>
+<label x="68.58" y="117.475" size="1.778" layer="95"/>
 </segment>
 </net>
@@
 </segment>
 <segment>
-<pinref part="P1" gate="G$1" pin="SU3"/>
-<wire x1="67.945" y1="162.56" x2="81.915" y2="162.56" width="0.1524" layer="91"/>
-<label x="67.945" y="163.195" size="1.778" layer="95"/>
+<pinref part="P1" gate="G$1" pin="SU5"/>
+<wire x1="67.945" y1="152.4" x2="81.915" y2="152.4" width="0.1524" layer="91"/>
+<label x="67.945" y="153.035" size="1.778" layer="95"/>
 </segment>
 </net>
